Commit message: This is a modified "struct.urdf" file

File: rob_struct/urdf/struct.urdf (robot description, URDF)
Before this commit: robot azi_bot, 8 links, 7 joints
Links:
- link gripper: geometry visual box size=0.1 0.1 0.1
Joints:
- removed joint gripper_joint

Commit message: This is wendessen, made change on the struct.urdf file

File: rob_struct/urdf/struct.urdf (robot description, URDF)
Before this commit: robot azi_bot, 7 links, 6 joints
Links:
- added link gripper
- link wheel_1: geometry visual cylinder length=0.05 radius=0.1
- link wheel_2: geometry visual cylinder length=0.05 radius=0.1
- link wheel_3: geometry visual cylinder length=0.05 radius=0.1
- link wheel_4: geometry visual cylinder length=0.05 radius=0.1
Joints:
- added joint gripper_joint: type continuous, parent box, child gripper, origin xyz=0.8 0.2 0.2 rpy=0 0 0
- joint wh1_joint: origin xyz=0.2 0 0 rpy=0 6.28 0 -> xyz=0.2 0 -0.1 rpy=0 6.28 0
- joint wh2_joint: origin xyz=0.8 0 0 rpy=0 6.28 0 -> xyz=0.8 0 -0.1 rpy=0 6.28 0
- joint wh3_joint: origin xyz=0.2 0.4 0 rpy=0 6.28 0 -> xyz=0.2 0.4 -0.1 rpy=0 6.28 0
- joint wh4_joint: origin xyz=0.8 0.4 0 rpy=0 6.28 0 -> xyz=0.8 0.4 -0.1 rpy=0 6.28 0

Commit message: This is a further modified urdf file

File: rob_struct/urdf/struct.urdf (robot description, URDF)
Before this commit: robot azi_bot, 8 links, 6 joints
Links:
- link gripper: geometry visual mesh filename=package://pr2_description/meshes/gripper_v0/l_finger.dae
Joints:
- added joint gripper_joint: type continuous, parent box, child gripper, origin xyz=0.9 0.2 0.2 rpy=0 0 0

Commit message: URDF

File: rob_struct/urdf/struct.urdf (robot description, URDF)
Before this commit: robot azi_bot, 8 links, 7 joints
Joints:
- joint camera_joint: limit (none) -> lower=-2.36 upper=2.36 effort=1000.0 velocity=0.5; type continuous -> revolute
- joint wh1_joint: origin xyz=0.2 0 -0.1 rpy=0 6.28 0 -> xyz=0.2 -0.05 0 rpy=0 6.28 0
- joint wh2_joint: origin xyz=0.8 0 -0.1 rpy=0 6.28 0 -> xyz=0.8 -0.05 0 rpy=0 6.28 0
- joint wh3_joint: origin xyz=0.2 0.4 -0.1 rpy=0 6.28 0 -> xyz=0.2 0.45 0 rpy=0 6.28 0
- joint wh4_joint: origin xyz=0.8 0.4 -0.1 rpy=0 6.28 0 -> xyz=0.8 0.45 0 rpy=0 6.28 0

Commit message: modified end effector

File: rob_struct/urdf/struct.urdf (robot description, URDF)
Before this commit: robot azi_bot, 8 links, 7 joints
Links:
- added link end_effector; visual mesh filename=package://pr2_description/meshes/gripper_v0/l_finger.dae
Joints:
- added joint end_joint: type revolute, parent gripper, child end_effector, origin xyz=0.2 0 0 rpy=0 0 0, limit lower=-2.36 upper=2.36 effort=1000.0 velocity=0.5
- joint camera_joint: limit (none) -> lower=-2.36 upper=2.36 effort=1000.0 velocity=0.5; type continuous -> revolute
- joint wh1_joint: origin xyz=0.2 0 -0.1 rpy=0 6.28 0 -> xyz=0.2 -0.05 0 rpy=0 6.28 0
- joint wh2_joint: origin xyz=0.8 0 -0.1 rpy=0 6.28 0 -> xyz=0.8 -0.05 0 rpy=0 6.28 0
- joint wh3_joint: origin xyz=0.2 0.4 -0.1 rpy=0 6.28 0 -> xyz=0.2 0.45 0 rpy=0 6.28 0
- joint wh4_joint: origin xyz=0.8 0.4 -0.1 rpy=0 6.28 0 -> xyz=0.8 0.45 0 rpy=0 6.28 0

Commit message: +launch

File: rob_struct/urdf/struct.urdf (robot description, URDF)
Before this commit: robot azi_bot, 9 links, 8 joints
Links:
- link camera: geometry visual mesh filename=package://rob_struct/meshes/kinect.dae scale=0.001 0.001 0.001
